File: untitled.brd (EAGLE design)
At the start: 75.9 x 49.5 mm, 13 parts

Commit message: second commit
Parts:
- added A+D1: (no value), connector:4P-2.54-80/40MIL
Connections:
- net +3V3: now also A+D1.3
- net GND: now also A+D1.4
- net IO32: now also A+D1.2
- net IO33: now also A+D1.1
Routing:
- net IO33: track 8.15 -> 32.3 mm
- net IO32: track 5.61 -> 27.2 mm
- net +3V3: track 67.3 -> 83.8 mm
- net GND: track 267.0 -> 275.9 mm
Changed lines of the file:
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@@
 <?xml version="1.0" encoding="utf-8"?>
 <!DOCTYPE eagle SYSTEM "eagle.dtd">
-<eagle version="8.5.2">
+<eagle version="8.4.3">
 <drawing>
 <settings>
@@
 <param name="checkRestrict" value="1"/>
 <param name="checkStop" value="0"/>
-<param name="checkValues" value="0"/>
 <param name="useDiameter" value="13"/>
 <param name="maxErrors" value="50"/>
@@
 <attribute name="VALUE" x="76.835" y="36.195" size="1.778" layer="21" ratio="10" rot="R90"/>
 </element>
+<element name="A+D1" library="connector" package="4P-2.54-80/40MIL" value="" x="55.88" y="40.64" smashed="yes">
+<attribute name="NAME" x="56.896" y="46.99" size="1.016" layer="25" rot="R180"/>
+<attribute name="VALUE" x="59.055" y="36.195" size="1.778" layer="21" ratio="10" rot="R90"/>
+</element>
 <element name="A+D4" library="connector" package="4P-2.54-80/40MIL" value="" x="55.88" y="24.13" smashed="yes">
 <attribute name="NAME" x="56.896" y="30.48" size="1.016" layer="25" rot="R180"/>
@@
 <contactref element="JP1" pad="13"/>
 <contactref element="JP1" pad="14"/>
+<contactref element="A+D1" pad="2"/>
+<wire x1="55.88" y1="41.91" x2="34.29" y2="41.91" width="0.254" layer="1"/>
 <wire x1="34.29" y1="41.91" x2="33.02" y2="40.64" width="0.254" layer="1"/>
 <wire x1="33.02" y1="40.64" x2="33.02" y2="39.37" width="0.254" layer="1"/>
@@
 <contactref element="JP1" pad="15"/>
 <contactref element="JP1" pad="16"/>
+<contactref element="A+D1" pad="1"/>
+<wire x1="55.88" y1="44.45" x2="31.75" y2="44.45" width="0.254" layer="1"/>
 <wire x1="31.75" y1="44.45" x2="30.48" y2="43.18" width="0.254" layer="1"/>
 <wire x1="30.48" y1="43.18" x2="30.48" y2="39.37" width="0.254" layer="1"/>
@@
 <contactref element="A+D2" pad="3"/>
 <contactref element="A+D3" pad="3"/>
+<contactref element="A+D1" pad="3"/>
 <contactref element="A+D4" pad="3"/>
 <contactref element="D1" pad="3"/>
@@
 <wire x1="48.26" y1="39.37" x2="48.26" y2="36.83" width="0.254" layer="1"/>
 <wire x1="73.66" y1="39.37" x2="64.77" y2="39.37" width="0.254" layer="1"/>
+<wire x1="64.77" y1="39.37" x2="55.88" y2="39.37" width="0.254" layer="1"/>
+<wire x1="55.88" y1="39.37" x2="48.26" y2="39.37" width="0.254" layer="1"/>
 <wire x1="64.77" y1="22.86" x2="59.69" y2="22.86" width="0.254" layer="1"/>
 <wire x1="59.69" y1="22.86" x2="55.88" y2="22.86" width="0.254" layer="1"/>
@@
 <via x="59.69" y="6.35" extent="1-16" drill="0.65"/>
 <wire x1="59.69" y1="22.86" x2="59.69" y2="6.35" width="0.254" layer="16"/>
-<wire x1="48.26" y1="39.37" x2="64.77" y2="39.37" width="0" layer="19" extent="1-1"/>
 </signal>
 <signal name="IO23">
@@
 <contactref element="A+D2" pad="4"/>
 <contactref element="A+D3" pad="4"/>
+<contactref element="A+D1" pad="4"/>
 <contactref element="A+D4" pad="4"/>
 <contactref element="A2V5" pad="4"/>
@@
 <wire x1="33.02" y1="11.43" x2="33.02" y2="8.89" width="0.254" layer="1"/>
 <wire x1="48.26" y1="11.43" x2="48.26" y2="8.89" width="0.254" layer="1"/>
+<wire x1="55.88" y1="36.83" x2="64.77" y2="36.83" width="0.254" layer="1"/>
 <wire x1="64.77" y1="36.83" x2="71.12" y2="36.83" width="0.254" layer="1"/>
 <wire x1="71.12" y1="36.83" x2="73.66" y2="36.83" width="0.254" layer="1"/>
