File: untitled.brd (EAGLE design)
At the start: 79.7 x 48.2 mm, 17 parts

Commit message: end of design
Parts:
- removed LOGO1: OSHW-LOGOMINI, SparkFun-Aesthetics:OSHW-LOGO-MINI
- removed LOGO2: ROHS_LOGO, SparkFun-Aesthetics:ROHS_LOGO_0.18_IN
- removed U$1: (no value), logo:CE_7.3MM
Routing:
- net GND: track 277.9 -> 205.6 mm, vias 5 -> 2
- net +3V3: track 91.2 -> 88.4 mm
Other:
- board size 79.7 x 48.2 mm -> 80.7 x 48.2 mm

Commit message: last commit
Routing:
- net +3V3: track 88.4 -> 86.6 mm, vias 3 -> 1
- net +5V: track 136.1 -> 135.4 mm, vias 3 -> 1
- net GND: vias 2 -> 1
Changed lines of the file:
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@@
 </signal>
 <signal name="+5V">
-<via x="69.85" y="7.62" extent="1-16" drill="0.65"/>
-<via x="69.85" y="24.13" extent="1-16" drill="0.65"/>
 <wire x1="49.53" y1="21.59" x2="49.53" y2="30.48" width="0.254" layer="16"/>
-<wire x1="69.85" y1="24.13" x2="69.85" y2="7.62" width="0.254" layer="16"/>
+<wire x1="69.85" y1="30.48" x2="69.85" y2="23" width="0.254" layer="16"/>
 <contactref element="JP1" pad="37"/>
 <contactref element="JP1" pad="38"/>
+<wire x1="69.85" y1="23" x2="69.85" y2="7.62" width="0.254" layer="16"/>
 <wire x1="2.54" y1="39.37" x2="2.54" y2="36.83" width="0.254" layer="1"/>
 <wire x1="2.54" y1="36.83" x2="2.54" y2="25.4" width="0.254" layer="1"/>
@@
 <contactref element="A2V5" pad="3"/>
 <contactref element="D2V5" pad="3"/>
-<wire x1="69.85" y1="24.13" x2="73.66" y2="24.13" width="0.254" layer="1"/>
-<wire x1="73.66" y1="24.13" x2="74.93" y2="23.13" width="0.254" layer="1"/>
-<wire x1="69.85" y1="30.48" x2="69.85" y2="24.13" width="0.254" layer="16"/>
 <wire x1="49.53" y1="30.48" x2="69.85" y2="30.48" width="0.254" layer="16"/>
-<wire x1="69.85" y1="7.62" x2="71.12" y2="6.35" width="0.254" layer="1"/>
-<wire x1="71.12" y1="6.35" x2="74.93" y2="6.35" width="0.254" layer="1"/>
-<wire x1="74.93" y1="6.35" x2="74.93" y2="6.62" width="0.254" layer="1"/>
 <wire x1="2.54" y1="39.37" x2="2.54" y2="41.91" width="0.254" layer="1"/>
 <wire x1="2.54" y1="41.91" x2="6.35" y2="45.72" width="0.254" layer="1"/>
+<wire x1="74.93" y1="6.62" x2="70.85" y2="6.62" width="0.254" layer="16"/>
+<wire x1="70.85" y1="6.62" x2="69.85" y2="7.62" width="0.254" layer="16"/>
+<wire x1="74.93" y1="23.13" x2="69.98" y2="23.13" width="0.254" layer="16"/>
+<wire x1="69.98" y1="23.13" x2="69.85" y2="23" width="0.254" layer="16"/>
 </signal>
 <signal name="TX">
@@
 <via x="48.26" y="22.86" extent="1-16" drill="0.65"/>
 <wire x1="48.26" y1="36.83" x2="48.26" y2="22.86" width="0.254" layer="16"/>
-<via x="59.69" y="24.13" extent="1-16" drill="0.65"/>
-<via x="59.69" y="7.35" extent="1-16" drill="0.65"/>
-<wire x1="59.69" y1="24.13" x2="59.69" y2="7.35" width="0.254" layer="16"/>
 <contactref element="A/D1" pad="3"/>
 <contactref element="A/D2" pad="3"/>
@@
 <contactref element="I2C" pad="3"/>
 <contactref element="D1" pad="3"/>
-<wire x1="57.15" y1="6.62" x2="60" y2="6.62" width="0.254" layer="1"/>
-<wire x1="60" y1="6.62" x2="66.04" y2="6.62" width="0.254" layer="1"/>
-<wire x1="57.15" y1="23.13" x2="58.42" y2="24.13" width="0.254" layer="1"/>
-<wire x1="58.42" y1="24.13" x2="59.69" y2="24.13" width="0.254" layer="1"/>
-<wire x1="59.69" y1="24.13" x2="64.77" y2="24.13" width="0.254" layer="1"/>
-<wire x1="64.77" y1="24.13" x2="66.04" y2="23.13" width="0.254" layer="1"/>
-<wire x1="59.69" y1="7.35" x2="59.69" y2="6.93" width="0.254" layer="1"/>
-<wire x1="59.69" y1="6.93" x2="60" y2="6.62" width="0.254" layer="1"/>
+<wire x1="57.15" y1="6.62" x2="60" y2="6.62" width="0.254" layer="16"/>
+<wire x1="60" y1="6.62" x2="66.04" y2="6.62" width="0.254" layer="16"/>
+<wire x1="57.15" y1="23.13" x2="60" y2="23.13" width="0.254" layer="16"/>
+<wire x1="60" y1="23.13" x2="66.04" y2="23.13" width="0.254" layer="16"/>
+<wire x1="60" y1="6.62" x2="60" y2="23.13" width="0.254" layer="16"/>
 </signal>
 <signal name="IO23">
@@
 <wire x1="33.02" y1="11.43" x2="33.02" y2="8.89" width="0.254" layer="1"/>
 <wire x1="48.26" y1="11.43" x2="48.26" y2="8.89" width="0.254" layer="1"/>
-<via x="48.26" y="20.32" extent="1-16" drill="0.65"/>
 <wire x1="50.8" y1="33.02" x2="68.58" y2="33.02" width="0.254" layer="16"/>
 <wire x1="50.8" y1="43.18" x2="50.8" y2="33.02" width="0.254" layer="16"/>
@@
 <contactref element="A/D4" pad="4"/>
 <contactref element="A1" pad="4"/>
-<wire x1="48.26" y1="20.32" x2="56.34" y2="20.32" width="0.254" layer="1"/>
-<wire x1="56.34" y1="20.32" x2="57.15" y2="21.13" width="0.254" layer="1"/>
 <wire x1="57.15" y1="21.13" x2="66.04" y2="21.13" width="0.254" layer="1"/>
 <contactref element="A2V5" pad="4"/>
@@
 <wire x1="48.26" y1="8.89" x2="52.53" y2="4.62" width="0.254" layer="16"/>
 <wire x1="52.53" y1="4.62" x2="57.15" y2="4.62" width="0.254" layer="16"/>
-<wire x1="48.26" y1="20.32" x2="48.26" y2="11.43" width="0.254" layer="16"/>
 <wire x1="33.02" y1="11.43" x2="34.59" y2="13" width="0.254" layer="16"/>
 <wire x1="47" y1="13" x2="48.26" y2="11.74" width="0.254" layer="16"/>
 <wire x1="48.26" y1="11.74" x2="48.26" y2="11.43" width="0.254" layer="16"/>
 <wire x1="34.59" y1="13" x2="47" y2="13" width="0.254" layer="16"/>
+<wire x1="48.26" y1="11.43" x2="48.26" y2="20.26" width="0.254" layer="16"/>
+<wire x1="49.13" y1="21.13" x2="57.15" y2="21.13" width="0.254" layer="16"/>
+<wire x1="48.26" y1="20.26" x2="49.13" y2="21.13" width="0.254" layer="16"/>
 </signal>
 <signal name="CRC">
