File: untitled.sch (EAGLE design)
At the start: 15 parts

Commit message: end of design
Parts:
- removed LOGO1: OSHW-LOGOMINI, SparkFun-Aesthetics:OSHW-LOGOMINI
- removed LOGO2: ROHS_LOGO, SparkFun-Aesthetics:ROHS_LOGO
Changed lines of the file:
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@@
 <part name="D1" library="Seeed-Connector -2016" deviceset="GROVE-CONNECTOR-DIP(4P-2.0)" device="" value="4P-2.0"/>
 <part name="D2V5" library="Seeed-Connector -2016" deviceset="GROVE-CONNECTOR-DIP(4P-2.0)" device="" value="4P-2.0"/>
-<part name="LOGO1" library="SparkFun-Aesthetics" library_urn="urn:adsk.eagle:library:507" deviceset="OSHW-LOGO" device="MINI" package3d_urn="urn:adsk.eagle:package:37101/1"/>
-<part name="LOGO2" library="SparkFun-Aesthetics" library_urn="urn:adsk.eagle:library:507" deviceset="ROHS_LOGO" device="" package3d_urn="urn:adsk.eagle:package:37159/1"/>
-<part name="LOGO3" library="logo" library_urn="urn:adsk.eagle:library:264" deviceset="CE_7.3MM" device=""/>
 </parts>
 <sheets>
@@
 <instance part="D1" gate="G$1" x="195.58" y="93.98"/>
 <instance part="D2V5" gate="G$1" x="220.98" y="93.98"/>
-<instance part="LOGO1" gate="G$1" x="205.74" y="35.56"/>
-<instance part="LOGO2" gate="G$1" x="223.52" y="25.4"/>
-<instance part="LOGO3" gate="G$1" x="246.38" y="25.4"/>
 </instances>
 <busses>
