File: untitled_v2.brd (EAGLE design)
At the start: 80.7 x 48.2 mm, 14 parts

Commit message: last commit
Parts:
- moved U$5 1.00 mm to (-1.27, 23.1)
Changed lines of the file:
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@@
 <setting verticaltext="up"/>
 </settings>
-<grid distance="1" unitdist="mm" unit="mm" style="lines" multiple="1" display="yes" altdistance="0.005" altunitdist="inch" altunit="inch"/>
+<grid distance="0.5" unitdist="mm" unit="mm" style="lines" multiple="1" display="yes" altdistance="0.005" altunitdist="inch" altunit="inch"/>
 <layers>
 <layer number="1" name="Top" color="4" fill="1" visible="yes" active="yes"/>
@@
 <attribute name="VALUE" x="49.53" y="14.605" size="1.27" layer="27" rot="R180"/>
 </element>
-<element name="U$5" library="SparkFun-Aesthetics" library_urn="urn:adsk.eagle:library:507" package="BREADBOARD_SPACING" package3d_urn="urn:adsk.eagle:package:37153/1" value="" x="-1.27" y="24.13" rot="R90"/>
+<element name="U$5" library="SparkFun-Aesthetics" library_urn="urn:adsk.eagle:library:507" package="BREADBOARD_SPACING" package3d_urn="urn:adsk.eagle:package:37153/1" value="" x="-1.27" y="23.13" rot="R90"/>
 <element name="R1" library="eagle-ltspice" library_urn="urn:adsk.eagle:library:217" package="0207/10" package3d_urn="urn:adsk.eagle:package:13275/1" value="1K" x="11.43" y="45.72" smashed="yes">
 <attribute name="SPICEMODEL" value="NONE" x="11.43" y="45.72" size="1.778" layer="27" display="off"/>

Commit message: first commit
Parts:
- removed A/D2, A/D3, A/D4, A1, A2V5, D1, D2V5: 4P-2.0, Seeed-Connector -2016:HW4-2.0
- removed JP1, JP2: (no value), pinhead:2X19
- removed LED: (no value), led:LED3MM
- removed R1: 1K, eagle-ltspice:0207/10
- added JP3: (no value), pinhead:1X12
- added JP4: (no value), pinhead:1X16
- added UART: 4P-2.0, Seeed-Connector -2016:HW4-2.0
- moved I2C 25.1 mm to (51.0, 32.0), turned to 0 degrees
- moved A/D1 18.2 mm to (54.1, 22.6)
- moved U$5 6.02 mm to (3.23, 27.1)
Connections:
- removed net +3V3: A/D1.3, A/D2.3, A/D3.3, A/D4.3, A1.3, D1.3, I2C.3, JP1.1, JP1.2
- removed net +5V: A2V5.3, D2V5.3, JP1.37, JP1.38, R1.1
- removed net CLK: JP2.37, JP2.38
- removed net CMD: JP1.35, JP1.36
- removed net CRC: LED.A, R1.2
- removed net IO0: JP2.27, JP2.28
- removed net IO16: D2V5.1, JP2.23, JP2.24
- removed net IO17: D2V5.2, JP2.21, JP2.22
- removed net IO18: D1.1, JP2.17, JP2.18
- removed net IO19: D1.2, JP2.15, JP2.16
- removed net IO2: JP2.29, JP2.30
- removed net IO21: I2C.2, JP2.11, JP2.12
- removed net IO22: I2C.1, JP2.5, JP2.6
- removed net IO23: JP2.3, JP2.4
- removed net IO25: A/D2.2, JP1.17, JP1.18
- removed net IO26: A/D2.1, JP1.19, JP1.20
- removed net IO34: A1.1, JP1.10, JP1.9
- removed net IO35: A1.2, JP1.11, JP1.12
- removed net IO4: A/D4.2, JP2.25, JP2.26
- removed net IO5: JP2.19, JP2.20
- removed net SD0: JP2.35, JP2.36
- removed net SD1: JP2.33, JP2.34
- removed net SD2: JP1.31, JP1.32
- removed net SD3: JP1.33, JP1.34
- removed net SVN: A2V5.2, JP1.7, JP1.8
- removed net SVP: A2V5.1, JP1.5, JP1.6
- new net 3V3: A/D1.3, I2C.3, JP4.2, UART.3
- new net A0: JP4.5
- new net A1: A/D1.1, JP4.6
- new net A2: A/D1.2, JP4.7
- new net A3: JP4.8
- new net A4: JP4.9
- new net A5: JP4.10
- new net ARF: JP4.3
- new net MISO: JP4.13
- new net MOSI: JP4.12
- new net RST: JP4.1
- new net SCK: JP4.11
- new net SCL: I2C.1, JP3.11
- new net SDA: I2C.2, JP3.12
- new net VBAT: JP3.1
- new net VBUS: JP3.3
- net EN: now also JP3.2; no longer JP1.3, JP1.4
- net GND: now also JP4.16, JP4.4, UART.4; no longer A/D2.4, A/D3.4, A/D4.4, A1.4, A2V5.4, D1.4, D2V5.4, JP1.27, JP1.28, JP2.1, JP2.13, JP2.14, JP2.2, LED.K
- net IO12: now also JP3.5; no longer JP1.25, JP1.26
- net IO13: now also JP3.4; no longer JP1.29, JP1.30
- net IO14: now also JP3.10; no longer A/D3.1, JP1.23, JP1.24
- net IO15: now also JP3.8; no longer A/D4.1, JP2.31, JP2.32
- net IO27: now also JP3.6; no longer A/D3.2, JP1.21, JP1.22
- net IO32: now also JP3.9; no longer A/D1.2, JP1.13, JP1.14
- net IO33: now also JP3.7; no longer A/D1.1, JP1.15, JP1.16
- net RX: now also JP4.14, UART.1; no longer JP2.10, JP2.9
- net TX: now also JP4.15, UART.2; no longer JP2.7, JP2.8
Routing:
- net GND: track 205.6 -> 0.00 mm, vias 1 -> 0
- net +5V: track 135.4 -> 0.00 mm, vias 1 -> 0
- net +3V3: track 86.6 -> 0.00 mm, vias 1 -> 0
- net IO15: track 67.2 -> 0.00 mm
- net IO16: track 65.4 -> 0.00 mm
- net IO14: track 63.2 -> 0.00 mm
- net IO17: track 63.0 -> 0.00 mm
- net IO27: track 61.2 -> 0.00 mm
- net IO4: track 53.0 -> 0.00 mm
- net IO26: track 50.3 -> 0.00 mm
- net IO25: track 47.2 -> 0.00 mm
- net SVN: track 46.1 -> 0.00 mm
- net IO18: track 45.6 -> 0.00 mm
- net IO19: track 42.9 -> 0.00 mm
- net IO35: track 42.3 -> 0.00 mm
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Other:
- board size 80.7 x 48.2 mm -> 57.2 x 33.8 mm
- board text removed: "IO14 IO27 3V3 GND"
- board text removed: "IO15 IO4 3V3 GND"
- board text removed: "IO16 IO17 5V GND"
- board text removed: "IO18 IO19 3V3 GND"
- board text removed: "IO22 IO21 3V3 GND"
- board text removed: "IO26 IO25 3V3 GND"
- board text removed: "IO34 IO35 3V3 GND"
- board text removed: "SVP SVN 5V GND"
