File: untitled_v2.sch (EAGLE design)
At the start: 13 parts

Commit message: first commit
Parts:
- removed A/D2, A/D3, A/D4, A1, A2V5, D1, D2V5: 4P-2.0, Seeed-Connector -2016:GROVE-CONNECTOR-DIP(4P-2.0)
- removed JP1, JP2: (no value), pinhead:PINHD-2X19
- removed LED: (no value), led:LED3MM
- removed R1: 1K, eagle-ltspice:R0207/10
- added JP3: (no value), pinhead:PINHD-1X12
- added JP4: (no value), pinhead:PINHD-1X16
- added UART: 4P-2.0, Seeed-Connector -2016:GROVE-CONNECTOR-DIP(4P-2.0)
Connections:
- removed net +3V3: A/D1.3, A/D2.3, A/D3.3, A/D4.3, A1.3, D1.3, I2C.3, JP1.1, JP1.2
- removed net +5V: A2V5.3, D2V5.3, JP1.37, JP1.38, R1.1
- removed net CLK: JP2.37, JP2.38
- removed net CMD: JP1.35, JP1.36
- removed net CRC: LED.A, R1.2
- removed net IO0: JP2.27, JP2.28
- removed net IO16: D2V5.1, JP2.23, JP2.24
- removed net IO17: D2V5.2, JP2.21, JP2.22
- removed net IO18: D1.1, JP2.17, JP2.18
- removed net IO19: D1.2, JP2.15, JP2.16
- removed net IO2: JP2.29, JP2.30
- removed net IO21: I2C.2, JP2.11, JP2.12
- removed net IO22: I2C.1, JP2.5, JP2.6
- removed net IO23: JP2.3, JP2.4
- removed net IO25: A/D2.2, JP1.17, JP1.18
- removed net IO26: A/D2.1, JP1.19, JP1.20
- removed net IO34: A1.1, JP1.10, JP1.9
- removed net IO35: A1.2, JP1.11, JP1.12
- removed net IO4: A/D4.2, JP2.25, JP2.26
- removed net IO5: JP2.19, JP2.20
- removed net SD0: JP2.35, JP2.36
- removed net SD1: JP2.33, JP2.34
- removed net SD2: JP1.31, JP1.32
- removed net SD3: JP1.33, JP1.34
- removed net SVN: A2V5.2, JP1.7, JP1.8
- removed net SVP: A2V5.1, JP1.5, JP1.6
- new net 3V3: A/D1.3, I2C.3, JP4.2, UART.3
- new net A0: JP4.5
- new net A1: A/D1.1, JP4.6
- new net A2: A/D1.2, JP4.7
- new net A3: JP4.8
- new net A4: JP4.9
- new net A5: JP4.10
- new net ARF: JP4.3
- new net MISO: JP4.13
- new net MOSI: JP4.12
- new net RST: JP4.1
- new net SCK: JP4.11
- new net SCL: I2C.1, JP3.11
- new net SDA: I2C.2, JP3.12
- new net VBAT: JP3.1
- new net VBUS: JP3.3
- net EN: now also JP3.2; no longer JP1.3, JP1.4
- net GND: now also JP4.16, JP4.4, UART.4; no longer A/D2.4, A/D3.4, A/D4.4, A1.4, A2V5.4, D1.4, D2V5.4, JP1.27, JP1.28, JP2.1, JP2.13, JP2.14, JP2.2, LED.C
- net IO12: now also JP3.5; no longer JP1.25, JP1.26
- net IO13: now also JP3.4; no longer JP1.29, JP1.30
- net IO14: now also JP3.10; no longer A/D3.1, JP1.23, JP1.24
- net IO15: now also JP3.8; no longer A/D4.1, JP2.31, JP2.32
- net IO27: now also JP3.6; no longer A/D3.2, JP1.21, JP1.22
- net IO32: now also JP3.9; no longer A/D1.2, JP1.13, JP1.14
- net IO33: now also JP3.7; no longer A/D1.1, JP1.15, JP1.16
- net RX: now also JP4.14, UART.1; no longer JP2.10, JP2.9
- net TX: now also JP4.15, UART.2; no longer JP2.7, JP2.8
Other:
- moved on the sheet: A/D1, I2C
