File: adalogger_shield_v1.brd (EAGLE design)
At the start: 49.2 x 24.8 mm, 6 parts

Commit message: dimensions ok
Parts:
- removed A/D1: 4P-2.0, Seeed-Connector -2016:HW4-2.0
- removed JP3: (no value), pinhead:1X12
- removed JP4: (no value), pinhead:1X16
- added A/D: 4P-2.0, Seeed-Connector -2016:HW4-2.0
- added JP1: (no value), microbuilder:1X12_ROUND
- added JP2: (no value), microbuilder:1X16_ROUND
- moved I2C 10.1 mm to (48.0, 23.0), turned to 90 degrees
- moved U$5 5.78 mm to (3.74, 21.4)
- moved UART 5.69 mm to (12.8, 23.0)
Connections:
- removed net 3V3: A/D1.3, I2C.3, JP4.2, UART.3
- new net 3V: A/D.2, I2C.2, JP2.15, UART.2
- net A0: now also JP2.12; no longer JP4.5
- net A1: now also A/D.4, JP2.11; no longer A/D1.1, JP4.6
- net A2: now also A/D.3, JP2.10; no longer A/D1.2, JP4.7
- net A3: now also JP2.9; no longer JP4.8
- net A4: now also JP2.8; no longer JP4.9
- net A5: now also JP2.7; no longer JP4.10
- net ARF: now also JP2.14; no longer JP4.3
- net EN: now also JP1.11; no longer JP3.2
- net GND: now also A/D.1, I2C.1, JP2.1, JP2.13, UART.1; no longer A/D1.4, I2C.4, JP4.16, JP4.4, UART.4
- net IO12: now also JP1.8; no longer JP3.5
- net IO13: now also JP1.9; no longer JP3.4
- net IO14: now also JP1.3; no longer JP3.10
- net IO15: now also JP1.5; no longer JP3.8
- net IO27: now also JP1.7; no longer JP3.6
- net IO32: now also JP1.4; no longer JP3.9
- net IO33: now also JP1.6; no longer JP3.7
- net MISO: now also JP2.4; no longer JP4.13
- net MOSI: now also JP2.5; no longer JP4.12
- net RST: now also JP2.16; no longer JP4.1
- net RX: now also JP2.3, UART.4; no longer JP4.14, UART.1
- net SCK: now also JP2.6; no longer JP4.11
- net SCL: now also I2C.4, JP1.2; no longer I2C.1, JP3.11
- net SDA: now also I2C.3, JP1.1; no longer I2C.2, JP3.12
- net TX: now also JP2.2, UART.3; no longer JP4.15, UART.2
- net VBAT: now also JP1.12; no longer JP3.1
- net VBUS: now also JP1.10; no longer JP3.3
Routing:
- net GND: track 0.00 -> 88.6 mm
- net TX: track 0.00 -> 65.5 mm
- net 3V: track 0.00 -> 49.7 mm
- net RX: track 0.00 -> 42.6 mm
- net A2: track 0.00 -> 12.1 mm
- net A1: track 0.00 -> 10.9 mm
- net SDA: track 0.00 -> 10.0 mm
- net SCL: track 0.00 -> 9.04 mm
- removed copper zone on layer 1, net GND
- removed copper zone on layer 16, net GND
Other:
- board size 49.2 x 24.8 mm -> 50.8 x 22.9 mm
- board text added: "10"
- board text added: "11"
- board text added: "12"
- board text added: "13"
- board text added: "3V"
- board text added: "5"
- board text added: "6"
- board text added: "9"
- board text added: "A/D"
- board text added: "A0"
- board text added: "A1"
- board text added: "A2"
- board text added: "A3"
- board text added: "A4"
- board text added: "A5"
- board text added: "ARf"
- board text added: "BAT"
- board text added: "EN"
- board text added: "GND"
- board text added: "GND 3V A2 A1"
- board text added: "GND 3V TX RX"
- board text added: "I2C"
- board text added: "MI"
- board text added: "MO"
- board text added: "NB-IoT Shield for Adafruit M0 Adalogger by www.thingforward.io"
- board text added: "RST"
- board text added: "RX"
- board text added: "SCK"
- board text added: "SCL"
- board text added: "SCL SDA 3V GND"
- board text added: "SDA"
- board text added: "TX"
- board text added: "UART"
- board text added: "USB"
- board text removed: "CLK SD0 SD1 IO15 IO17 IO5 IO18 IO19 GND IO21 RXD TXD IO22 IO23 GND"
- board text removed: "Grove Base Shield for ESP32-DevKitC by ThingForward www.thingforward.io"
- board text removed: "IO33 IO32 3V3 GND"
- board text removed: "V5 CMD SD3 SD2 IO13 GND IO26 IO25 SVN SVP EN 3V3"

Commit message: routing ok
Parts:
- added A/D2: 4P-2.0, Seeed-Connector -2016:HW4-2.0
- moved A/D 20.9 mm to (9.62, 21.4)
- moved UART 7.15 mm to (14.8, 29.8), turned to 180 degrees
- moved I2C 3.64 mm to (51.3, 21.4)
Connections:
- net 3V: now also A/D2.2
- net A3: now also A/D2.4
- net A4: now also A/D2.3
- net GND: now also A/D2.1
Routing:
- net TX: track 65.5 -> 43.9 mm
- net A3: track 0.00 -> 14.7 mm
- net GND: track 88.6 -> 75.7 mm
- net A4: track 0.00 -> 12.5 mm
- net 3V: track 49.7 -> 61.6 mm
- net A2: track 12.1 -> 20.5 mm
- net A1: track 10.9 -> 18.1 mm
- net SCL: track 9.04 -> 11.3 mm
- net SDA: track 10.0 -> 11.6 mm
- net RX: track 42.6 -> 43.5 mm, vias 0 -> 1
Other:
- board text added: "A/D2"
- board text added: "A3 A4 GND 3V"
- board text added: "NB-IoT Shield for Adafruit M0 Adalogger www.thingforward.io"
- board text removed: "NB-IoT Shield for Adafruit M0 Adalogger by www.thingforward.io"
