File: adalogger_shield_v1.brd (EAGLE design)
At the start: 50.8 x 22.9 mm, 7 parts

Commit message: test ok
Parts:
- removed U$5: (no value), SparkFun-Aesthetics:BREADBOARD_SPACING
- moved JP1 12.3 mm to (30.2, 21.8)
- moved UART 12.3 mm to (9.76, 18.6)
- moved A/D 12.3 mm to (4.54, 10.3)
- moved A/D2 12.3 mm to (30.2, 10.3)
- moved I2C 12.3 mm to (46.2, 10.3)
- moved JP2 12.3 mm to (25.1, 1.52)
Other:
- board text added: "NB-IoT Shield for Adafruit Boards by www.thingforward.io"
- board text removed: "A3 A4 GND 3V"
- board text removed: "GND 3V A2 A1"
- board text removed: "GND 3V TX RX"
- board text removed: "NB-IoT Shield for Adafruit M0 Adalogger www.thingforward.io"
- board text removed: "SCL SDA 3V GND"
