File: adalogger_shield_v1.brd (EAGLE design)
At the start: 50.8 x 22.9 mm, 6 parts

Commit message: second version OK
Parts:
- removed A/D2: 4P-2.0, Seeed-Connector -2016:HW4-2.0
- moved UART 23.1 mm to (31.7, 11.4), turned to 90 degrees
- moved A/D 3.50 mm to (7.84, 11.4), turned to 90 degrees
- moved I2C 3.50 mm to (42.9, 11.4), turned to 270 degrees
- moved JP1 0.25 mm to (30.2, 21.6)
- moved JP2 0.25 mm to (25.1, 1.27)
Connections:
- net 3V: now also A/D.3, I2C.3, UART.3; no longer A/D.2, A/D2.2, I2C.2, UART.2
- net A1: now also A/D.1; no longer A/D.4
- net A2: now also A/D.2; no longer A/D.3
- net A3: no longer A/D2.4
- net A4: no longer A/D2.3
- net GND: now also A/D.4, I2C.4, UART.4; no longer A/D.1, A/D2.1, I2C.1, UART.1
- net RX: now also UART.1; no longer UART.4
- net SCL: now also I2C.1; no longer I2C.4
- net SDA: now also I2C.2; no longer I2C.3
- net TX: now also UART.2; no longer UART.3
Routing:
- net RX: track 43.5 -> 10.9 mm, vias 1 -> 0
- net GND: track 75.7 -> 45.3 mm
- net TX: track 43.9 -> 13.9 mm
- net A3: track 14.7 -> 0.00 mm
- net 3V: track 61.6 -> 47.3 mm
- net A4: track 12.5 -> 0.00 mm
- net A1: track 18.1 -> 14.2 mm
- net SCL: track 11.3 -> 7.67 mm
- net A2: track 20.5 -> 17.6 mm
Other:
- board text removed: "A/D2"
