File: adalogger_shield_v1.sch (EAGLE design)
At the start: 5 parts

Commit message: dimensions ok
Parts:
- removed JP3: (no value), pinhead:PINHD-1X12
- removed JP4: (no value), pinhead:PINHD-1X16
- added JP1: (no value), microbuilder:HEADER-1X12
- added JP2: (no value), microbuilder:HEADER-1X16ROUND
- renumbered A/D1 to A/D
Connections:
- removed net 3V3: A/D.3, I2C.3, JP4.2, UART.3
- new net 3V: A/D.2, I2C.2, JP2.15, UART.2
- net A0: now also JP2.12; no longer JP4.5
- net A1: now also A/D.4, JP2.11; no longer A/D.1, JP4.6
- net A2: now also A/D.3, JP2.10; no longer A/D.2, JP4.7
- net A3: now also JP2.9; no longer JP4.8
- net A4: now also JP2.8; no longer JP4.9
- net A5: now also JP2.7; no longer JP4.10
- net ARF: now also JP2.14; no longer JP4.3
- net EN: now also JP1.11; no longer JP3.2
- net GND: now also A/D.1, I2C.1, JP2.1, JP2.13, UART.1; no longer A/D.4, I2C.4, JP4.16, JP4.4, UART.4
- net IO12: now also JP1.8; no longer JP3.5
- net IO13: now also JP1.9; no longer JP3.4
- net IO14: now also JP1.3; no longer JP3.10
- net IO15: now also JP1.5; no longer JP3.8
- net IO27: now also JP1.7; no longer JP3.6
- net IO32: now also JP1.4; no longer JP3.9
- net IO33: now also JP1.6; no longer JP3.7
- net MISO: now also JP2.4; no longer JP4.13
- net MOSI: now also JP2.5; no longer JP4.12
- net RST: now also JP2.16; no longer JP4.1
- net RX: now also JP2.3, UART.4; no longer JP4.14, UART.1
- net SCK: now also JP2.6; no longer JP4.11
- net SCL: now also I2C.4, JP1.2; no longer I2C.1, JP3.11
- net SDA: now also I2C.3, JP1.1; no longer I2C.2, JP3.12
- net TX: now also JP2.2, UART.3; no longer JP4.15, UART.2
- net VBAT: now also JP1.12; no longer JP3.1
- net VBUS: now also JP1.10; no longer JP3.3

Commit message: routing ok
Parts:
- added A/D2: 4P-2.0, Seeed-Connector -2016:GROVE-CONNECTOR-DIP(4P-2.0)
Connections:
- net 3V: now also A/D2.2
- net A3: now also A/D2.4
- net A4: now also A/D2.3
- net GND: now also A/D2.1
Changed lines of the file:
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@@
 <part name="GND2" library="supply1" library_urn="urn:adsk.eagle:library:371" deviceset="GND" device=""/>
 <part name="GND1" library="supply1" library_urn="urn:adsk.eagle:library:371" deviceset="GND" device=""/>
+<part name="A/D2" library="Seeed-Connector -2016" deviceset="GROVE-CONNECTOR-DIP(4P-2.0)" device="" value="4P-2.0"/>
+<part name="GND3" library="supply1" library_urn="urn:adsk.eagle:library:371" deviceset="GND" device=""/>
 </parts>
 <sheets>
@@
 <instance part="GND2" gate="1" x="180.34" y="121.92" rot="R180"/>
 <instance part="GND1" gate="1" x="180.34" y="96.52" rot="R180"/>
+<instance part="A/D2" gate="G$1" x="220.98" y="114.3"/>
+<instance part="GND3" gate="1" x="210.82" y="121.92" rot="R180"/>
 </instances>
 <busses>
@@
 <wire x1="180.34" y1="92.71" x2="180.34" y2="93.98" width="0.1524" layer="91"/>
 </segment>
+<segment>
+<pinref part="A/D2" gate="G$1" pin="1"/>
+<pinref part="GND3" gate="1" pin="GND"/>
+<wire x1="217.17" y1="118.11" x2="210.82" y2="118.11" width="0.1524" layer="91"/>
+<wire x1="210.82" y1="118.11" x2="210.82" y2="119.38" width="0.1524" layer="91"/>
+</segment>
 </net>
 <net name="RST" class="0">
@@
 <pinref part="JP2" gate="A" pin="9"/>
 </segment>
+<segment>
+<pinref part="A/D2" gate="G$1" pin="4"/>
+<wire x1="217.17" y1="110.49" x2="210.82" y2="110.49" width="0.1524" layer="91"/>
+<label x="205.74" y="109.22" size="1.778" layer="95"/>
+</segment>
 </net>
 <net name="A4" class="0">
@@
 <pinref part="JP2" gate="A" pin="8"/>
 </segment>
+<segment>
+<pinref part="A/D2" gate="G$1" pin="3"/>
+<wire x1="217.17" y1="113.03" x2="210.82" y2="113.03" width="0.1524" layer="91"/>
+<label x="205.74" y="111.76" size="1.778" layer="95"/>
+</segment>
 </net>
 <net name="A5" class="0">
@@
 <label x="175.26" y="88.9" size="1.778" layer="95"/>
 </segment>
-</net>
+<segment>
+<pinref part="A/D2" gate="G$1" pin="2"/>
+<wire x1="217.17" y1="115.57" x2="210.82" y2="115.57" width="0.1524" layer="91"/>
+<label x="205.74" y="114.3" size="1.778" layer="95"/>
+</segment>
+</net>
