File: adalogger_shield_v1.sch (EAGLE design)
At the start: 6 parts

Commit message: second version OK
Parts:
- removed A/D2: 4P-2.0, Seeed-Connector -2016:GROVE-CONNECTOR-DIP(4P-2.0)
Connections:
- net 3V: now also A/D.3, I2C.3, UART.3; no longer A/D.2, A/D2.2, I2C.2, UART.2
- net A1: now also A/D.1; no longer A/D.4
- net A2: now also A/D.2; no longer A/D.3
- net A3: no longer A/D2.4
- net A4: no longer A/D2.3
- net GND: now also A/D.4, I2C.4, UART.4; no longer A/D.1, A/D2.1, I2C.1, UART.1
- net RX: now also UART.1; no longer UART.4
- net SCL: now also I2C.1; no longer I2C.4
- net SDA: now also I2C.2; no longer I2C.3
- net TX: now also UART.2; no longer UART.3
